File: Batman-dock.kicad_pcb (KiCad board)
At the start: 2 copper layers, 40 x 12 mm, 5 parts, among them J1 TYPECL324LBCP24, J2 70AAJL6LM0G, J3 70AAJL6LM0G

Commit message: Backplate push on PCB.  Backplate insertion tolerance.
Other:
- board text added: "Rev. ${REVISION} Batman-dock"
- board text removed: "Batman-dock Rev. ${REVISION}"
Changed lines of the file:
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@@
 	(paper "A4")
 	(title_block
-		(rev "B")
+		(rev "C")
 	)
 	(layers
@@
 		(layer "Edge.Cuts")
 	)
-	(gr_text "Batman-dock\nRev. ${REVISION}"
-		(at 142.855 93.42 0)
+	(gr_text "Rev. ${REVISION}\nBatman-dock"
+		(at 141.4 98.16 0)
 		(layer "B.SilkS")
 		(effects
